File: schematics/MindBrain/mindbrain_schematic_v2.brd (EAGLE design)
At the start: 81 x 47.6 mm, 51 parts, among them CON1 POWER, IC1 TL084, IC2 TL084

Commit message: cleaned up schematic thx nathan
Connections:
- net N$25 renamed +12V
- net N$27 renamed -12V
Routing:
- net -12V: track 81.9 -> 0.00 mm
- net +12V: track 81.2 -> 0.00 mm
- net GND: track 12.7 -> 0.00 mm
Changed lines of the file:
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@@
 <contactref element="RIN8" pad="P$1"/>
 <contactref element="R8" pad="P$1"/>
-<contactref element="CON1" pad="6"/>
-<contactref element="CON1" pad="4"/>
-<contactref element="CON1" pad="8"/>
-<contactref element="CON1" pad="7"/>
-<contactref element="CON1" pad="3"/>
-<contactref element="CON1" pad="5"/>
 <contactref element="C2" pad="2"/>
 <contactref element="C4" pad="2"/>
 <contactref element="C1" pad="2"/>
 <contactref element="C3" pad="2"/>
-<wire x1="5.08" y1="22.225" x2="7.62" y2="22.225" width="0.4064" layer="1"/>
-<wire x1="5.08" y1="27.305" x2="7.62" y2="27.305" width="0.4064" layer="1"/>
-<wire x1="5.08" y1="24.765" x2="7.62" y2="24.765" width="0.4064" layer="1"/>
 <contactref element="AUDIOCARD-GND" pad="1"/>
 <contactref element="OUTPUT-GND" pad="1"/>
 <contactref element="AUDIOCARD-GND1" pad="1"/>
 <contactref element="OUTPUT-GND1" pad="1"/>
-<wire x1="7.62" y1="27.305" x2="7.62" y2="22.225" width="0.4064" layer="1"/>
 <polygon width="0.4064" layer="16">
 <vertex x="-0.3175" y="47.9425"/>
@@
 <vertex x="-0.3175" y="47.9425"/>
 </polygon>
+<contactref element="CON1" pad="7"/>
+<contactref element="CON1" pad="3"/>
+<contactref element="CON1" pad="5"/>
+<contactref element="CON1" pad="8"/>
+<contactref element="CON1" pad="4"/>
+<contactref element="CON1" pad="6"/>
 </signal>
 <signal name="N$2">
@@
 <wire x1="27.94" y1="29.845" x2="27.94" y2="28.575" width="0.4064" layer="1"/>
 </signal>
-<signal name="N$27">
+<signal name="N$26">
+<via x="16.51" y="42.545" extent="1-16" drill="0.6"/>
+</signal>
+<signal name="N$28">
+<via x="71.12" y="10.795" extent="1-16" drill="0.6"/>
+</signal>
+<signal name="N$29">
+<via x="45.72" y="29.845" extent="1-16" drill="0.6"/>
+</signal>
+<signal name="N$30">
+<via x="45.72" y="19.685" extent="1-16" drill="0.6"/>
+</signal>
+<signal name="-12V">
 <contactref element="CON1" pad="1"/>
 <contactref element="CON1" pad="2"/>
+<contactref element="C2" pad="1"/>
 <contactref element="IC1" pad="11"/>
 <contactref element="IC2" pad="11"/>
-<contactref element="C2" pad="1"/>
 <contactref element="C4" pad="1"/>
-<wire x1="5.08" y1="29.845" x2="7.62" y2="29.845" width="0.4064" layer="1"/>
-<wire x1="7.62" y1="29.845" x2="7.62" y2="36.195" width="0.4064" layer="16"/>
-<wire x1="7.62" y1="36.195" x2="10.16" y2="38.735" width="0.4064" layer="16"/>
-<wire x1="10.16" y1="38.735" x2="27.94" y2="38.735" width="0.4064" layer="16"/>
-<wire x1="27.94" y1="38.735" x2="31.877" y2="34.798" width="0.4064" layer="16"/>
-<wire x1="31.877" y1="34.798" x2="33.02" y2="34.798" width="0.4064" layer="16"/>
-<wire x1="33.02" y1="28.575" x2="33.02" y2="34.798" width="0.4064" layer="16"/>
-<wire x1="58.42" y1="29.21" x2="58.42" y2="28.575" width="0.4064" layer="16"/>
-<wire x1="58.42" y1="28.575" x2="58.42" y2="34.798" width="0.4064" layer="16"/>
-<wire x1="58.42" y1="28.575" x2="58.42" y2="34.925" width="0.4064" layer="16"/>
-<wire x1="58.42" y1="34.925" x2="58.293" y2="34.798" width="0.4064" layer="16"/>
-<wire x1="58.293" y1="34.798" x2="33.02" y2="34.798" width="0.4064" layer="16"/>
-</signal>
-<signal name="N$25">
+<wire x1="58.42" y1="28.575" x2="58.42" y2="34.798" width="0" layer="19" extent="1-1"/>
+<wire x1="33.02" y1="34.798" x2="58.42" y2="34.798" width="0" layer="19" extent="1-1"/>
+<wire x1="33.02" y1="28.575" x2="33.02" y2="34.798" width="0" layer="19" extent="1-1"/>
+<wire x1="7.62" y1="29.845" x2="33.02" y2="28.575" width="0" layer="19" extent="1-1"/>
+<wire x1="5.08" y1="29.845" x2="7.62" y2="29.845" width="0" layer="19" extent="1-1"/>
+</signal>
+<signal name="+12V">
+<contactref element="CON1" pad="10"/>
+<contactref element="CON1" pad="9"/>
+<contactref element="C1" pad="1"/>
 <contactref element="IC1" pad="4"/>
-<contactref element="C1" pad="1"/>
-<contactref element="CON1" pad="9"/>
+<contactref element="C3" pad="1"/>
 <contactref element="IC2" pad="4"/>
-<contactref element="C3" pad="1"/>
-<contactref element="CON1" pad="10"/>
-<wire x1="5.08" y1="19.685" x2="7.62" y2="19.685" width="0.4064" layer="1"/>
-<wire x1="7.62" y1="19.685" x2="7.62" y2="13.335" width="0.4064" layer="16"/>
-<wire x1="7.62" y1="13.335" x2="10.16" y2="10.795" width="0.4064" layer="16"/>
-<wire x1="10.16" y1="10.795" x2="27.94" y2="10.795" width="0.4064" layer="16"/>
-<wire x1="27.94" y1="10.795" x2="31.877" y2="14.732" width="0.4064" layer="16"/>
-<wire x1="31.877" y1="14.732" x2="33.02" y2="14.732" width="0.4064" layer="16"/>
-<wire x1="33.02" y1="14.732" x2="33.02" y2="20.955" width="0.4064" layer="16"/>
-<wire x1="58.42" y1="14.732" x2="58.42" y2="20.955" width="0.4064" layer="16"/>
-<wire x1="33.02" y1="20.955" x2="33.02" y2="14.605" width="0.4064" layer="16"/>
-<wire x1="33.02" y1="14.605" x2="33.147" y2="14.732" width="0.4064" layer="16"/>
-<wire x1="33.147" y1="14.732" x2="58.42" y2="14.732" width="0.4064" layer="16"/>
-</signal>
-<signal name="N$26">
-<via x="16.51" y="42.545" extent="1-16" drill="0.6"/>
-</signal>
-<signal name="N$28">
-<via x="71.12" y="10.795" extent="1-16" drill="0.6"/>
-</signal>
-<signal name="N$29">
-<via x="45.72" y="29.845" extent="1-16" drill="0.6"/>
-</signal>
-<signal name="N$30">
-<via x="45.72" y="19.685" extent="1-16" drill="0.6"/>
+<wire x1="58.42" y1="14.732" x2="58.42" y2="20.955" width="0" layer="19" extent="1-1"/>
+<wire x1="33.02" y1="20.955" x2="58.42" y2="20.955" width="0" layer="19" extent="1-1"/>
+<wire x1="33.02" y1="14.732" x2="33.02" y2="20.955" width="0" layer="19" extent="1-1"/>
+<wire x1="7.62" y1="19.685" x2="33.02" y2="20.955" width="0" layer="19" extent="1-1"/>
+<wire x1="5.08" y1="19.685" x2="7.62" y2="19.685" width="0" layer="19" extent="1-1"/>
 </signal>
 </signals>

Commit message: Passing DRC and ERC!!!
Routing:
- net +12V: track 0.00 -> 81.6 mm
- net -12V: track 0.00 -> 81.0 mm
Changed lines of the file:
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@@
 <setting verticaltext="up"/>
 </settings>
-<grid distance="0.025" unitdist="inch" unit="inch" style="lines" multiple="1" display="no" altdistance="0.0125" altunitdist="inch" altunit="inch"/>
+<grid distance="0.025" unitdist="inch" unit="inch" style="lines" multiple="1" display="yes" altdistance="0.0125" altunitdist="inch" altunit="inch"/>
 <layers>
 <layer number="1" name="Top" color="4" fill="1" visible="yes" active="yes"/>
@@
 2016</text>
 <text x="3.175" y="38.1" size="1.27" layer="21" font="vector">-12V</text>
-<text x="77.47" y="36.195" size="1.016" layer="21">GND</text>
-<text x="77.47" y="33.655" size="1.016" layer="21">GND</text>
-<text x="76.835" y="31.115" size="1.016" layer="21">OUT8</text>
-<text x="76.835" y="28.575" size="1.016" layer="21">OUT7</text>
-<text x="76.835" y="26.035" size="1.016" layer="21">OUT6</text>
-<text x="76.835" y="23.495" size="1.016" layer="21">OUT5</text>
-<text x="76.835" y="20.955" size="1.016" layer="21">OUT4</text>
-<text x="76.835" y="18.415" size="1.016" layer="21">OUT3</text>
-<text x="76.835" y="15.875" size="1.016" layer="21">OUT2</text>
-<text x="76.835" y="13.335" size="1.016" layer="21">OUT1</text>
-<text x="18.415" y="36.195" size="1.016" layer="21">GND</text>
-<text x="18.415" y="33.655" size="1.016" layer="21">GND</text>
-<text x="18.415" y="31.115" size="1.016" layer="21">IN8</text>
-<text x="18.415" y="28.575" size="1.016" layer="21">IN7</text>
-<text x="18.415" y="26.035" size="1.016" layer="21">IN6</text>
-<text x="18.415" y="23.495" size="1.016" layer="21">IN5</text>
-<text x="18.415" y="20.955" size="1.016" layer="21">IN4</text>
-<text x="18.415" y="18.415" size="1.016" layer="21">IN3</text>
-<text x="18.415" y="15.875" size="1.016" layer="21">IN2</text>
-<text x="18.415" y="13.335" size="1.016" layer="21">IN1</text>
+<text x="19.05" y="35.8775" size="0.8128" layer="21">GND</text>
+<text x="19.05" y="33.3375" size="0.8128" layer="21">GND</text>
+<text x="76.835" y="35.8775" size="0.8128" layer="21">GND</text>
+<text x="76.835" y="33.3375" size="0.8128" layer="21">GND</text>
+<text x="19.05" y="30.7975" size="0.8128" layer="21">IN8</text>
+<text x="19.05" y="28.2575" size="0.8128" layer="21">IN7</text>
+<text x="19.05" y="25.7175" size="0.8128" layer="21">IN6</text>
+<text x="19.05" y="23.1775" size="0.8128" layer="21">IN5</text>
+<text x="19.05" y="20.6375" size="0.8128" layer="21">IN4</text>
+<text x="19.05" y="18.0975" size="0.8128" layer="21">IN3</text>
+<text x="19.05" y="15.5575" size="0.8128" layer="21">IN2</text>
+<text x="19.05" y="13.0175" size="0.8128" layer="21">IN1</text>
+<text x="76.835" y="30.7975" size="0.8128" layer="21">OUT8</text>
+<text x="76.835" y="28.2575" size="0.8128" layer="21">OUT7</text>
+<text x="76.835" y="25.7175" size="0.8128" layer="21">OUT6</text>
+<text x="76.835" y="23.1775" size="0.8128" layer="21">OUT5</text>
+<text x="76.835" y="20.6375" size="0.8128" layer="21">OUT4</text>
+<text x="76.835" y="18.0975" size="0.8128" layer="21">OUT3</text>
+<text x="76.835" y="15.5575" size="0.8128" layer="21">OUT2</text>
+<text x="76.835" y="13.0175" size="0.8128" layer="21">OUT1</text>
 </plain>
 <attributes>
@@
 <contactref element="IC2" pad="11"/>
 <contactref element="C4" pad="1"/>
-<wire x1="58.42" y1="28.575" x2="58.42" y2="34.798" width="0" layer="19" extent="1-1"/>
-<wire x1="33.02" y1="34.798" x2="58.42" y2="34.798" width="0" layer="19" extent="1-1"/>
-<wire x1="33.02" y1="28.575" x2="33.02" y2="34.798" width="0" layer="19" extent="1-1"/>
-<wire x1="7.62" y1="29.845" x2="33.02" y2="28.575" width="0" layer="19" extent="1-1"/>
-<wire x1="5.08" y1="29.845" x2="7.62" y2="29.845" width="0" layer="19" extent="1-1"/>
+<wire x1="7.62" y1="29.845" x2="5.08" y2="29.845" width="0.4064" layer="16"/>
+<wire x1="7.62" y1="29.845" x2="7.62" y2="30.48" width="0.4064" layer="16"/>
+<wire x1="7.62" y1="30.48" x2="15.875" y2="38.735" width="0.4064" layer="16"/>
+<wire x1="15.875" y1="38.735" x2="29.083" y2="38.735" width="0.4064" layer="16"/>
+<wire x1="29.083" y1="38.735" x2="33.02" y2="34.798" width="0.4064" layer="16"/>
+<wire x1="33.02" y1="28.575" x2="33.02" y2="34.798" width="0.4064" layer="16"/>
+<wire x1="58.42" y1="28.575" x2="58.42" y2="34.798" width="0.4064" layer="16"/>
+<wire x1="58.42" y1="28.575" x2="58.42" y2="34.925" width="0.4064" layer="16"/>
+<wire x1="58.42" y1="34.925" x2="57.785" y2="34.925" width="0.4064" layer="16"/>
+<wire x1="57.785" y1="34.925" x2="53.975" y2="38.735" width="0.4064" layer="16"/>
+<wire x1="53.975" y1="38.735" x2="36.957" y2="38.735" width="0.4064" layer="16"/>
+<wire x1="36.957" y1="38.735" x2="33.02" y2="34.798" width="0.4064" layer="16"/>
 </signal>
 <signal name="+12V">
@@
 <contactref element="C3" pad="1"/>
 <contactref element="IC2" pad="4"/>
-<wire x1="58.42" y1="14.732" x2="58.42" y2="20.955" width="0" layer="19" extent="1-1"/>
-<wire x1="33.02" y1="20.955" x2="58.42" y2="20.955" width="0" layer="19" extent="1-1"/>
-<wire x1="33.02" y1="14.732" x2="33.02" y2="20.955" width="0" layer="19" extent="1-1"/>
-<wire x1="7.62" y1="19.685" x2="33.02" y2="20.955" width="0" layer="19" extent="1-1"/>
-<wire x1="5.08" y1="19.685" x2="7.62" y2="19.685" width="0" layer="19" extent="1-1"/>
+<wire x1="7.62" y1="19.685" x2="5.08" y2="19.685" width="0.4064" layer="16"/>
+<wire x1="7.62" y1="19.685" x2="7.62" y2="19.05" width="0.4064" layer="16"/>
+<wire x1="7.62" y1="19.05" x2="15.875" y2="10.795" width="0.4064" layer="16"/>
+<wire x1="15.875" y1="10.795" x2="29.083" y2="10.795" width="0.4064" layer="16"/>
+<wire x1="29.083" y1="10.795" x2="33.02" y2="14.732" width="0.4064" layer="16"/>
+<wire x1="33.02" y1="14.732" x2="33.02" y2="20.955" width="0.4064" layer="16"/>
+<wire x1="58.42" y1="14.732" x2="58.42" y2="20.955" width="0.4064" layer="16"/>
+<wire x1="33.02" y1="20.955" x2="33.02" y2="14.605" width="0.4064" layer="16"/>
+<wire x1="33.02" y1="14.605" x2="37.465" y2="10.16" width="0.4064" layer="16"/>
+<wire x1="37.465" y1="10.16" x2="53.848" y2="10.16" width="0.4064" layer="16"/>
+<wire x1="53.848" y1="10.16" x2="58.42" y2="14.732" width="0.4064" layer="16"/>
 </signal>
 </signals>
